Commit message: Imported upstream version '1.1.3' of 'upstream'

File: vs060/model/vs060A1_AV6_NNN_NNN.urdf (robot description, URDF)
Before this commit: robot vs060A1_AV6_NNN_NNN, 7 links, 6 joints
Links:
- added link base_link
Joints:
- added joint base_link_joint: type fixed, parent base_link, child BASE
